File: eagle projects/ADCS Sensor Board/SensorBoard.sch (EAGLE design)
At the start: 95 parts, among them J5 HDR_10_EZFET_DEBUGGER, J6 MTI-1_8428-11B1-RK-TP, Q1 BC850SMD, Q2 IRF7507TRPBF, U1 MSP430F5529IPN, U2 LMV321, U3 ADS7841E_2K5, U4 LMV321, U6 LMV321, Y1 32.768kHz, Y2 CSTCR4M00G15L99

Commit message: Renumbered parts and exported bom CSV
Parts:
- removed C26: 0.1u, rcl:C-EUC0603
- removed C27: 1n, rcl:C-EUC0805
- removed C28: 470n, rcl:C-EUC0805
- removed R100: 0R, rcl:R-US_R0805
- removed R53, R55: 1k, rcl:R-US_R0402
- removed R54, R56: 2k, rcl:R-US_R0402
- added C11: 0.1u, rcl:C-EUC0603
- added C8: 100n, rcl:C-EUC0402
- added C9: 1u, resistor:C-EUC1206
- added R26: 5.6k, rcl:R-US_R0805
- added R32: 750R, rcl:R-US_R0603
- added R33, R34, R35: 0R, rcl:R-US_R0805
- C10: value 1n -> 0.1u; device rcl:C-EUC0402 -> rcl:C-EUC0603
- C13: value 0.1u -> 1u; device rcl:C-EUC0603 -> resistor:C-EUC1206
- C15, C16: value 1u -> 0.1u; device resistor:C-EUC1206 -> rcl:C-EUC0603
- C17, C23: value 0.1u -> 1n; device rcl:C-EUC0603 -> rcl:C-EUC0805
- C18: value 0.1u -> 1n; device rcl:C-EUC0603 -> resistor:C-EUC1206
- C20: value 1n -> 0.1u; device rcl:C-EUC0805 -> rcl:C-EUC0603
- C21: device resistor:C-EUC1206 -> rcl:C-EUC0805
- C24: value 1n -> 470n
- C3: value 100n -> 12p
- C5: value 12p -> 100n
- C7: value 100n -> 1n
- JP1: device my_library:JP1Q_ -> my_library:PINHD-1X4
- JP4: device my_library:PINHD-2X6 -> my_library:PINHD-1X4
- JP5: device my_library:PINHD-1X4 -> my_library:PINHD-2X6
- JP6: device my_library:PINHD-1X3 -> my_library:JP1Q_
- JP9: device my_library:PINHD-1X4 -> my_library:PINHD-1X3
- R10, R17: value 5.6k -> 1k
- R11, R18, R24, R25: value 1.37M -> 1k
- R12: value 1.37M -> 5.6k
- R13, R20, R21: value 1k -> 5.6k
- R14: value 1k -> 1.37M
- R15: value 5.1M -> 1.37M; device resistor:R-US_R1206 -> rcl:R-US_R0805
- R16: value 5.6k -> 0R
- R19: value 1.37M -> 5.1M; device rcl:R-US_R0805 -> resistor:R-US_R1206
- R2: value 47k -> 1k
- R22, R23: value 5.6k -> 1.37M
- R27: value 27R -> 5.6k
- R28: value 0R -> 1.37M
- R29: value 470R -> 1.37M; device rcl:R-US_R0603 -> rcl:R-US_R0805
- R3: value 0R -> 2k; device rcl:R-US_R0805 -> rcl:R-US_R0402
- R30: value 470R -> 27R; device rcl:R-US_R0603 -> rcl:R-US_R0805
- R31: value 750R -> 470R
- R4: value 0R -> 1k; device rcl:R-US_R0805 -> rcl:R-US_R0402
- R5: value 1M -> 2k
- R6: value 200R -> 1M; device resistor:R-US_R1206 -> rcl:R-US_R0402
- R7: value 1k -> 47k; device rcl:R-US_R0805 -> rcl:R-US_R0402
- R8: value 1k -> 470R; device rcl:R-US_R0805 -> rcl:R-US_R0603
- R9: value 5.6k -> 200R; device rcl:R-US_R0805 -> resistor:R-US_R1206
- renumbered J5 to J1, J6 to J2, U6 to U5
Connections:
- net !CS!_SUN_Z+: now also JP1.2; no longer JP9.2
- net !CS!_SUN_Z-: now also JP4.2; no longer JP8.2
- net !RST!_MTI: now also TP3.TP; no longer TP5.TP
- net +3V3: now also C11.1, C13.1, C20.1, C5.2, C8.1, C9.1, JP5.1, JP8.2, R10.1, R17.1, R24.1, R31.1, R7.2, R9.2; no longer C17.1, C18.1, C23.1, C26.1, C3.2, C7.1, JP4.1, JP5.2, R13.1, R2.2, R20.1, R27.1, R6.2, R7.1
- net +5V: now also JP8.1, R2.2, R32.1; no longer JP5.1, R31.1, R53.2
- net ACT_BRD_3V_PRESENT: now also JP5.7; no longer JP4.7
- net ACT_BRD_5V_PRESENT: now also R4.2; no longer R55.2
- net ACT_BRD_5V_SHIFTED: now also JP5.5, R4.1, R5.2; no longer JP4.5, R55.1, R56.2
- net B_MEAS_X: now also C21.2, R23.1; no longer C24.2, R19.1
- net B_MEAS_Y: now also C17.2, R15.1; no longer C20.2, R12.1
- net B_MEAS_Z: now also C23.2, R29.1; no longer C27.2, R25.1
- net GND: now also C10.1, C11.2, C13.2, C20.2, C24.1, C8.2, C9.2, JP8.4, R11.2, R18.2, R19.1, R25.2, R3.1, R6.1; no longer C10.2, C13.1, C17.2, C18.2, C23.2, C26.2, C28.1, JP5.4, R14.2, R15.1, R21.2, R54.1, R56.1, R8.2
- net INIT_EPS_BURN_WIRE: now also JP8.3; no longer JP5.3
- net MSP430_ACTIVE: now also JP5.10, R8.1; no longer JP4.10, R29.1
- net MSP_OBC_RESET: now also JP5.9; no longer JP4.9
- net MTI_DRDY: now also TP5.TP; no longer TP3.TP
- net N$1: now also JP9.1, R33.2; no longer JP6.1, R28.2
- net N$2: now also JP9.2, R34.2; no longer JP6.2, R4.2
- net N$20: now also R10.2, R14.1; no longer R7.2, R8.1
- net N$21: now also C17.1, R13.1, R15.2; no longer C20.1, R10.1, R12.2
- net N$23: now also R12.1, R14.2; no longer R11.2, R9.1
- net N$3: now also JP9.3, R35.2; no longer JP6.3, R3.2
- net N$35: now also C18.2, JP6.2, R16.1; no longer C21.2, JP1.2, R100.1
- net N$36: now also R19.2; no longer R15.2
- net N$37: now also JP6.1, R16.2; no longer JP1.1, R100.2
- net N$38: now also C18.1; no longer C21.1
- net N$39: now also C10.2, R9.1; no longer C13.2, R6.1
- net N$4: now also R8.2; no longer R29.2
- net N$49: now also R17.2, R22.1; no longer R13.2, R14.1
- net N$5: now also R31.2; no longer R30.2
- net N$50: now also C21.1, R21.1, R23.2; no longer C24.1, R17.1, R19.2
- net N$52: now also R20.1, R22.2; no longer R16.1, R18.2
- net N$59: now also R24.2, R25.1, R28.1; no longer R20.2, R21.1, R24.1
- net N$6: now also R32.2; no longer R31.2
- net N$60: now also C23.1, R27.1, R29.2; no longer C27.1, R23.1, R25.2
- net N$62: now also R26.1, R28.2; no longer R22.1, R24.2
- net N$7: now also C24.2, R30.2; no longer C28.2, R27.2
- net OUT_A_N: now also R12.2; no longer R9.2
- net OUT_A_P: now also R13.2; no longer R10.2
- net OUT_B_N: now also R20.2; no longer R16.2
- net OUT_B_P: now also R21.2; no longer R17.2
- net OUT_C_N: now also R26.2; no longer R22.2
- net OUT_C_P: now also R27.2; no longer R23.2
- net P5.4/XIN1: now also C3.2; no longer C4.2
- net P5.5/XOUT1: now also C4.2; no longer C5.2
- net RESERVED_1: now also JP5.2; no longer JP4.2
- net RESERVED_2: now also JP5.4; no longer JP4.4
- net RESERVED_3: now also JP5.6; no longer JP4.6
- net RESERVED_4: now also JP5.8; no longer JP4.8
- net RST/SBWTDIO: now also C7.1, R7.1; no longer C10.1, R2.1
- net SEN_BRD_5V_PRESENT: now also JP5.3, R2.1, R3.2; no longer JP4.3, R53.1, R54.2
- net TARGET_PUR: now also R6.2; no longer R5.2
- net UCA0RXD: now also JP5.12; no longer JP4.12
- net UCA0TXD: now also JP5.11; no longer JP4.11
- net UCB0_SPI_CLK: now also JP1.1, JP4.1, R33.1; no longer JP8.1, JP9.1, R28.1
- net UCB0_SPI_MISO: now also JP1.4, JP4.4, R34.1; no longer JP8.4, JP9.4, R4.1
- net UCB0_SPI_MOSI: now also JP1.3, JP4.3, R35.1; no longer JP8.3, JP9.3, R3.1
Other:
- moved on the sheet: C12, C13, C14, C15, C16, C17, C18, C19, C20, C21, C22, C23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
