File: eagle projects/ADCS Actuator Board/ActuatorBoard.sch (EAGLE design)
At the start: 290 parts, among them J19 TE_1-84953-1, J20 TE_1-84953-1, J21 TE_1-84953-1, U1 TVS991, U10 DRV10970_MOTOR_DRIVERDRV10970, U12 DRV10970_MOTOR_DRIVERDRV10970, U13 ADS7841E_2K5, U15 TLV9051IDCKR, U19 TLV9051IDCKR, U2 ADS7841E_2K5, U21 TLV9051IDCKR, U23 TLV9051IDCKR, U24 TLV9051IDCKR, U25 ADS7841E_2K5, U26 TLV9051IDCKR, U27 ADS7841E_2K5, U28 TLV9051IDCKR, U29 TLV9051IDCKR, U3 ADS7841E_2K5, U30 TLV9051IDCKR, U31 TLV9051IDCKR, U32 TLV9051IDCKR, U35 BD6210F-E2, U39 BD6210F-E2, U4 ADS7841E_2K5, U5 TVS991, U6 TLV9051IDCKR, U7 DRV10970_MOTOR_DRIVERDRV10970, U8 TVS991, U9 BD6210F-E2

Commit message: Removed the godawful sun sensing circuitry
Parts:
- removed C100, C101, C105, C110, C111, C115, C116, C54, C70, C71, C84, C98: 0.022u, resistor:C-EUC0402
- removed C102, C104, C107, C109, C112, C114, C46, C48, C49, C51, C53, C65, C67, C69, C73, C75, C76, C78, C79, C81, C83, C86, C88, C90, C92, C93, C95, C97: 0.1u, resistor:C-EUC0402
- removed C103, C106, C108, C113, C52, C55, C68, C82, C85, C87, C96, C99: 4.7u, resistor:C-EUC0402
- removed C28, C45, C47, C50, C66, C72, C74, C77, C80, C89, C91, C94: 1u, resistor:C-EUC0402
- removed J10, J11, J12, J13, J14, J15, J16, J17, J18, J7, J8, J9: (no value), my_library:TRM_BLK_1X2
- removed R22, R25, R32, R38, R44, R50, R53, R56, R59, R62, R65, R68: 280R, resistor:R-US_R0402
- removed R23, R28, R33, R39, R45, R51, R54, R57, R60, R63, R66, R69: 13.7k, resistor:R-US_R0402
- removed R24, R31, R34, R40, R46, R52, R55, R58, R61, R64, R67, R70: 3.74k, resistor:R-US_R0402
- removed R3, R4, R5, R6: 10k, rcl:R-US_R0402
- removed TP1, TP10, TP11, TP12, TP13, TP14, TP15, TP16, TP17, TP18, TP19, TP20, TP3, TP6, TP8, TP9: TESTPOINT, my_library:TESTPOINT
- removed U13, U25, U27, U4: ADS7841E_2K5, my_library:ADS7841E_2K5
- removed U15, U19, U21, U23, U24, U26, U28, U29, U30, U31, U32, U6: TLV9051IDCKR, my_library:TLV9051IDCKR
Connections:
- removed net N$1: TP1.TP, U13.CH0
- removed net N$2: TP9.TP, U25.CH0
- removed net N$22: C51.1, R4.1, U13.!SHDN
- removed net N$23: C100.1, J7.2, R31.1, U23.-
- removed net N$24: C81.1, R6.1, U4.!SHDN
- removed net N$25: C95.1, R5.1, U27.!SHDN
- removed net N$29: C84.1, J8.2, R24.1, U6.-
- removed net N$3: TP13.TP, U27.CH0
- removed net N$31: R22.2, R23.1, U6.+
- removed net N$34: R25.2, R28.1, U23.+
- removed net N$35: C101.1, J9.2, R34.1, U24.-
- removed net N$36: R32.2, R33.1, U24.+
- removed net N$37: C98.1, J12.2, R64.1, U30.-
- removed net N$38: C54.1, J15.2, R40.1, U15.-
- removed net N$4: C102.1, R3.1, U25.!SHDN
- removed net N$41: R38.2, R39.1, U15.+
- removed net N$44: C70.1, J14.2, R46.1, U19.-
- removed net N$45: R44.2, R45.1, U19.+
- removed net N$46: C71.1, J13.2, R52.1, U21.-
- removed net N$47: R50.2, R51.1, U21.+
- removed net N$49: C105.1, J18.2, R55.1, U26.-
- removed net N$54: R53.2, R54.1, U26.+
- removed net N$55: C110.1, J17.2, R58.1, U28.-
- removed net N$56: R56.2, R57.1, U28.+
- removed net N$57: C111.1, J16.2, R61.1, U29.-
- removed net N$58: R59.2, R60.1, U29.+
- removed net N$61: R62.2, R63.1, U30.+
- removed net N$63: C115.1, J11.2, R67.1, U31.-
- removed net N$64: R65.2, R66.1, U31.+
- removed net N$65: C116.1, J10.2, R70.1, U32.-
- removed net N$66: R68.2, R69.1, U32.+
- removed net N$9: TP17.TP, U4.CH0
- removed net X+_0_DEGREES: C105.2, R55.2, TP14.TP, U25.CH1, U26.OUT
- removed net X+_120_DEGREES: C110.2, R58.2, TP15.TP, U25.CH2, U28.OUT
- removed net X+_240_DEGREES: C111.2, R61.2, TP16.TP, U25.CH3, U29.OUT
- removed net X-_0_DEGREES: C54.2, R40.2, TP10.TP, U13.CH1, U15.OUT
- removed net X-_120_DEGREES: C70.2, R46.2, TP11.TP, U13.CH2, U19.OUT
- removed net X-_240_DEGREES: C71.2, R52.2, TP12.TP, U13.CH3, U21.OUT
- removed net Y+_0_DEGREES: C98.2, R64.2, TP18.TP, U27.CH1, U30.OUT
- removed net Y+_120_DEGREES: C115.2, R67.2, TP19.TP, U27.CH2, U31.OUT
- removed net Y+_240_DEGREES: C116.2, R70.2, TP20.TP, U27.CH3, U32.OUT
- removed net Y-_0_DEGREES: C84.2, R24.2, TP3.TP, U4.CH1, U6.OUT
- removed net Y-_120_DEGREES: C100.2, R31.2, TP6.TP, U23.OUT, U4.CH2
- removed net Y-_240_DEGREES: C101.2, R34.2, TP8.TP, U24.OUT, U4.CH3
- net !CS!_SUN_X+: no longer U25.!CS
- net !CS!_SUN_X-: no longer U13.!CS
- net !CS!_SUN_Y+: no longer U27.!CS
- net !CS!_SUN_Y-: no longer U4.!CS
- net +3V3: no longer C103.1, C104.1, C106.1, C107.1, C108.1, C109.1, C112.1, C113.1, C114.1, C28.1, C45.1, C46.1, C47.1, C48.1, C49.1, C50.1, C52.1, C53.1, C55.1, C65.1, C66.1, C67.1, C68.1, C69.1, C72.1, C73.1, C74.1, C75.1, C76.1, C77.1, C78.1, C79.1, C80.1, C82.1, C83.1, C85.1, C86.1, C87.1, C88.1, C89.1, C90.1, C91.1, C92.1, C93.1, C94.1, C96.1, C97.1, C99.1, R23.2, R28.2, R3.2, R33.2, R39.2, R4.2, R45.2, R5.2, R51.2, R54.2, R57.2, R6.2, R60.2, R63.2, R66.2, R69.2, U13.VCC+, U13.VCC+_2, U13.VREF, U15.V+, U19.V+, U21.V+, U23.V+, U24.V+, U25.VCC+, U25.VCC+_2, U25.VREF, U26.V+, U27.VCC+, U27.VCC+_2, U27.VREF, U28.V+, U29.V+, U30.V+, U31.V+, U32.V+, U4.VCC+, U4.VCC+_2, U4.VREF, U6.V+
- net GND: no longer C102.2, C103.2, C104.2, C106.2, C107.2, C108.2, C109.2, C112.2, C113.2, C114.2, C28.2, C45.2, C46.2, C47.2, C48.2, C49.2, C50.2, C51.2, C52.2, C53.2, C55.2, C65.2, C66.2, C67.2, C68.2, C69.2, C72.2, C73.2, C74.2, C75.2, C76.2, C77.2, C78.2, C79.2, C80.2, C81.2, C82.2, C83.2, C85.2, C86.2, C87.2, C88.2, C89.2, C90.2, C91.2, C92.2, C93.2, C94.2, C95.2, C96.2, C97.2, C99.2, J10.1, J11.1, J12.1, J13.1, J14.1, J15.1, J16.1, J17.1, J18.1, J7.1, J8.1, J9.1, R22.1, R25.1, R32.1, R38.1, R44.1, R50.1, R53.1, R56.1, R59.1, R62.1, R65.1, R68.1, U13.COM, U13.GND, U13.MODE, U15.V-, U19.V-, U21.V-, U23.V-, U24.V-, U25.COM, U25.GND, U25.MODE, U26.V-, U27.COM, U27.GND, U27.MODE, U28.V-, U29.V-, U30.V-, U31.V-, U32.V-, U4.COM, U4.GND, U4.MODE, U6.V-
- net UCB0_SPI_CLK: no longer U13.DCLK, U25.DCLK, U27.DCLK, U4.DCLK
- net UCB0_SPI_MISO: no longer U13.DOUT, U25.DOUT, U27.DOUT, U4.DOUT
- net UCB0_SPI_MOSI: no longer U13.DIN, U25.DIN, U27.DIN, U4.DIN

Commit message: Sanity check
Parts:
- R26, R27: value 500R -> 470R
Connections:
- removed net !CS!_SUN_X+: J2.16
- removed net !CS!_SUN_X-: J2.14
- removed net !CS!_SUN_Y+: J2.3
- removed net !CS!_SUN_Y-: J2.1
Other:
- note added: "3-Pin header Jumper on this Rev for testing both mode configurations"
- note added: "3V3 Present Signal"
- note added: "5V Present Signal"
- note added: "Hall sensors on Maxon motor require external pull-up resistor"
- note added: "Only X and Y magnetorquer mounted physically to board"
- note added: "Only Z-axis Reaction wheel mounted physically to PCB"
