File: eagle projects/ADCS Actuator Board/ActuatorBoard.sch (EAGLE design)
At the start: 153 parts, among them J19 TE_1-84953-1, J20 TE_1-84953-1, J21 TE_1-84953-1, U1 TVS991, U10 DRV10970_MOTOR_DRIVERDRV10970, U12 DRV10970_MOTOR_DRIVERDRV10970, U2 ADS7841E_2K5, U3 ADS7841E_2K5, U35 BD6210F-E2, U39 BD6210F-E2, U5 TVS991, U7 DRV10970_MOTOR_DRIVERDRV10970, U8 TVS991, U9 BD6210F-E2

Commit message: bfwebfibc
Parts:
- added R45, R46: 5.1M, rcl:R-US_R0402
Connections:
- new net N$1: R45.1, U2.BUSY
- new net N$2: R46.2, U3.BUSY
- net GND: now also R45.2, R46.1
Other:
- note added: "J. Smith, T. Christison"
- moved on the sheet: C23, C43, R14
Changed lines of the file:
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@@
 <part name="P+19" library="supply1" library_urn="urn:adsk.eagle:library:371" deviceset="+5V" device=""/>
 <part name="P+20" library="supply1" library_urn="urn:adsk.eagle:library:371" deviceset="+5V" device=""/>
+<part name="R45" library="rcl" library_urn="urn:adsk.eagle:library:334" deviceset="R-US_" device="R0402" package3d_urn="urn:adsk.eagle:package:23547/3" value="5.1M"/>
+<part name="SUPPLY40" library="supply2" library_urn="urn:adsk.eagle:library:372" deviceset="GND" device=""/>
+<part name="R46" library="rcl" library_urn="urn:adsk.eagle:library:334" deviceset="R-US_" device="R0402" package3d_urn="urn:adsk.eagle:package:23547/3" value="5.1M"/>
+<part name="SUPPLY47" library="supply2" library_urn="urn:adsk.eagle:library:372" deviceset="GND" device=""/>
 </parts>
 <sheets>
@@
 <text x="127" y="132.08" size="1.778" layer="97">Only X and Y magnetorquer mounted
 physically to board</text>
+<text x="190.5" y="11.43" size="2.54" layer="94">J. Smith, T. Christison</text>
 </plain>
 <instances>
@@
 <attribute name="VALUE" x="127.635" y="9.525" size="1.778" layer="96"/>
 </instance>
-<instance part="C43" gate="G$1" x="137.16" y="22.86" smashed="yes">
-<attribute name="NAME" x="140.97" y="20.955" size="1.778" layer="95"/>
-<attribute name="VALUE" x="140.716" y="18.669" size="1.778" layer="96"/>
+<instance part="C43" gate="G$1" x="139.7" y="22.86" smashed="yes">
+<attribute name="NAME" x="143.51" y="20.955" size="1.778" layer="95"/>
+<attribute name="VALUE" x="143.256" y="18.669" size="1.778" layer="96"/>
 </instance>
 <instance part="R13" gate="G$1" x="144.78" y="25.4" smashed="yes">
@@
 <attribute name="VALUE" x="146.05" y="28.702" size="1.778" layer="96" rot="R180"/>
 </instance>
-<instance part="SUPPLY116" gate="GND" x="137.16" y="12.7" smashed="yes">
-<attribute name="VALUE" x="135.255" y="9.525" size="1.778" layer="96"/>
+<instance part="SUPPLY116" gate="GND" x="139.7" y="12.7" smashed="yes">
+<attribute name="VALUE" x="137.795" y="9.525" size="1.778" layer="96"/>
 </instance>
 <instance part="+3V61" gate="G$1" x="40.64" y="33.02" smashed="yes">
@@
 <attribute name="VALUE" x="229.87" y="83.82" size="1.778" layer="96" rot="R180"/>
 </instance>
+<instance part="R45" gate="G$1" x="147.32" y="5.08" smashed="yes">
+<attribute name="NAME" x="143.51" y="9.1186" size="1.778" layer="95"/>
+<attribute name="VALUE" x="148.59" y="8.382" size="1.778" layer="96" rot="R180"/>
+</instance>
+<instance part="SUPPLY40" gate="GND" x="154.94" y="5.08" smashed="yes" rot="R90">
+<attribute name="VALUE" x="158.115" y="3.175" size="1.778" layer="96" rot="R90"/>
+</instance>
 </instances>
 <busses>
@@
 <pinref part="SUPPLY116" gate="GND" pin="GND"/>
 <pinref part="C43" gate="G$1" pin="2"/>
-<wire x1="137.16" y1="15.24" x2="137.16" y2="17.78" width="0.1524" layer="91"/>
+<wire x1="139.7" y1="15.24" x2="139.7" y2="17.78" width="0.1524" layer="91"/>
 </segment>
 <segment>
@@
 <pinref part="SUPPLY23" gate="GND" pin="GND"/>
 </segment>
+<segment>
+<pinref part="R45" gate="G$1" pin="2"/>
+<pinref part="SUPPLY40" gate="GND" pin="GND"/>
+</segment>
 </net>
 <net name="+5V" class="0">
@@
 <pinref part="C43" gate="G$1" pin="1"/>
 <pinref part="R13" gate="G$1" pin="1"/>
-<wire x1="137.16" y1="25.4" x2="139.7" y2="25.4" width="0.1524" layer="91"/>
 <pinref part="U2" gate="A" pin="!SHDN"/>
-<wire x1="137.16" y1="25.4" x2="127" y2="25.4" width="0.1524" layer="91"/>
-<junction x="137.16" y="25.4"/>
+<wire x1="139.7" y1="25.4" x2="127" y2="25.4" width="0.1524" layer="91"/>
+<junction x="139.7" y="25.4"/>
 </segment>
 </net>
@@
 </segment>
 </net>
+<net name="N$1" class="0">
+<segment>
+<pinref part="U2" gate="A" pin="BUSY"/>
+<wire x1="127" y1="22.86" x2="134.62" y2="22.86" width="0.1524" layer="91"/>
+<wire x1="134.62" y1="22.86" x2="134.62" y2="5.08" width="0.1524" layer="91"/>
+<pinref part="R45" gate="G$1" pin="1"/>
+<wire x1="142.24" y1="5.08" x2="134.62" y2="5.08" width="0.1524" layer="91"/>
+</segment>
+</net>
 </nets>
 </sheet>
@@
 <wire x1="91.44" y1="50.8" x2="91.44" y2="20.32" width="0.1524" layer="97" grouprefs="BD621F-EF_LOGIC_TABLE"/>
 <wire x1="40.64" y1="45.72" x2="124.46" y2="45.72" width="0.1524" layer="97" style="shortdash" grouprefs="BD621F-EF_LOGIC_TABLE"/>
+<text x="191.77" y="11.43" size="2.54" layer="94">J. Smith, T. Christison</text>
 </plain>
 <instances>
@@
 <text x="17.78" y="22.86" size="1.778" layer="97">3-Pin header Jumper on this Rev for
 testing both mode configurations</text>
+<text x="191.77" y="11.43" size="2.54" layer="94">J. Smith, T. Christison</text>
 </plain>
 <instances>
@@
 <text x="175.26" y="208.28" size="1.778" layer="97">Hall sensors on Maxon motor require external pull-up resistor</text>
 <text x="68.58" y="200.66" size="1.778" layer="97">Only Z-axis Reaction wheel mounted physically to PCB</text>
+<text x="191.77" y="11.43" size="2.54" layer="94">J. Smith, T. Christison</text>
 </plain>
 <instances>
@@
 <attribute name="VALUE" x="122.555" y="103.505" size="1.778" layer="96"/>
 </instance>
-<instance part="C23" gate="G$1" x="132.08" y="116.84" smashed="yes">
-<attribute name="NAME" x="135.89" y="114.935" size="1.778" layer="95"/>
-<attribute name="VALUE" x="135.636" y="112.649" size="1.778" layer="96"/>
-</instance>
-<instance part="R14" gate="G$1" x="139.7" y="119.38" smashed="yes">
-<attribute name="NAME" x="135.89" y="123.4186" size="1.778" layer="95"/>
-<attribute name="VALUE" x="140.97" y="122.682" size="1.778" layer="96" rot="R180"/>
+<instance part="C23" gate="G$1" x="134.62" y="116.84" smashed="yes">
+<attribute name="NAME" x="138.43" y="114.935" size="1.778" layer="95"/>
+<attribute name="VALUE" x="138.176" y="112.649" size="1.778" layer="96"/>
+</instance>
+<instance part="R14" gate="G$1" x="144.78" y="119.38" smashed="yes">
+<attribute name="NAME" x="140.97" y="123.4186" size="1.778" layer="95"/>
+<attribute name="VALUE" x="146.05" y="122.682" size="1.778" layer="96" rot="R180"/>
 </instance>
-<instance part="SUPPLY33" gate="GND" x="132.08" y="106.68" smashed="yes">
-<attribute name="VALUE" x="130.175" y="103.505" size="1.778" layer="96"/>
+<instance part="SUPPLY33" gate="GND" x="134.62" y="106.68" smashed="yes">
+<attribute name="VALUE" x="132.715" y="103.505" size="1.778" layer="96"/>
 </instance>
 <instance part="+3V60" gate="G$1" x="33.02" y="127" smashed="yes">
 <attribute name="VALUE" x="35.56" y="129.54" size="1.778" layer="96" rot="R180"/>
 </instance>
-<instance part="+3V65" gate="G$1" x="144.78" y="127" smashed="yes">
-<attribute name="VALUE" x="147.32" y="129.54" size="1.778" layer="96" rot="R180"/>
+<instance part="+3V65" gate="G$1" x="149.86" y="127" smashed="yes">
+<attribute name="VALUE" x="152.4" y="129.54" size="1.778" layer="96" rot="R180"/>
 </instance>
 <instance part="SUPPLY34" gate="GND" x="53.34" y="111.76" smashed="yes">
@@
 <attribute name="VALUE" x="142.748" y="50.8" size="1.778" layer="96" rot="R270"/>
 </instance>
+<instance part="R46" gate="G$1" x="129.54" y="99.06" smashed="yes" rot="R90">
+<attribute name="NAME" x="125.5014" y="95.25" size="1.778" layer="95" rot="R90"/>
+<attribute name="VALUE" x="126.238" y="100.33" size="1.778" layer="96" rot="R270"/>
+</instance>
+<instance part="SUPPLY47" gate="GND" x="129.54" y="91.44" smashed="yes">
+<attribute name="VALUE" x="127.635" y="88.265" size="1.778" layer="96"/>
+</instance>
 </instances>
 <busses>
@@
 <pinref part="SUPPLY33" gate="GND" pin="GND"/>
 <pinref part="C23" gate="G$1" pin="2"/>
-<wire x1="132.08" y1="109.22" x2="132.08" y2="111.76" width="0.1524" layer="91"/>
+<wire x1="134.62" y1="109.22" x2="134.62" y2="111.76" width="0.1524" layer="91"/>
 </segment>
 <segment>
@@
 <wire x1="67.31" y1="81.28" x2="66.04" y2="81.28" width="0.1524" layer="91"/>
 </segment>
+<segment>
+<pinref part="R46" gate="G$1" pin="1"/>
+<pinref part="SUPPLY47" gate="GND" pin="GND"/>
+</segment>
 </net>
 <net name="Z_HALL_B" class="0">
@@
 <segment>
 <pinref part="R14" gate="G$1" pin="2"/>
-<wire x1="144.78" y1="119.38" x2="144.78" y2="124.46" width="0.1524" layer="91"/>
+<wire x1="149.86" y1="119.38" x2="149.86" y2="124.46" width="0.1524" layer="91"/>
 <pinref part="+3V65" gate="G$1" pin="+3V3"/>
 </segment>
@@
 <pinref part="C23" gate="G$1" pin="1"/>
 <pinref part="R14" gate="G$1" pin="1"/>
-<wire x1="132.08" y1="119.38" x2="134.62" y2="119.38" width="0.1524" layer="91"/>
+<wire x1="134.62" y1="119.38" x2="139.7" y2="119.38" width="0.1524" layer="91"/>
 <pinref part="U3" gate="A" pin="!SHDN"/>
-<wire x1="132.08" y1="119.38" x2="121.92" y2="119.38" width="0.1524" layer="91"/>
-<junction x="132.08" y="119.38"/>
+<wire x1="134.62" y1="119.38" x2="121.92" y2="119.38" width="0.1524" layer="91"/>
+<junction x="134.62" y="119.38"/>
 </segment>
 </net>
@@
 </segment>
 </net>
+<net name="N$2" class="0">
+<segment>
+<pinref part="U3" gate="A" pin="BUSY"/>
+<wire x1="121.92" y1="116.84" x2="129.54" y2="116.84" width="0.1524" layer="91"/>
+<wire x1="129.54" y1="104.14" x2="129.54" y2="116.84" width="0.1524" layer="91"/>
+<pinref part="R46" gate="G$1" pin="2"/>
+</segment>
+</net>

Commit message: Last commit before major layout changes on Actuator board Rev B
Parts:
- removed J2, J3: (no value), my_library:PINHD-2X8_TXT-MOVED
- added J7: CNC_3221-10-0300-00, my_library:CNC_3221-10-0300-00
- added J8: CNC_3221-14-0300-00, my_library:CNC_3221-14-0300-00
Connections:
- removed net !CS!_CUR_SENSE_MAG: J2.11, U2.!CS
- removed net !CS!_CUR_SENSE_RW: J2.13, U3.!CS
- new net !CS!_CURR_SENSE_MTQR: J7.5, U2.!CS
- new net !CS!_CURR_SENSE_RW: J7.3, U3.!CS
- new net MAG_Y_FIN\: J8.6
- new net N$37: J7.10
- new net N$42: J7.9
- net +3V3: now also J7.7; no longer J2.15
- net +5V: now also J8.14; no longer J3.14
- net MAG_X_FIN: now also J8.10; no longer J3.10
- net MAG_X_RIN: now also J8.12; no longer J3.12
- net MAG_Y_FIN: no longer J3.6
- net MAG_Y_RIN: now also J8.8; no longer J3.8
- net MAG_Z_FIN: now also J8.2; no longer J3.2
- net MAG_Z_RIN: now also J8.4; no longer J3.4
- net RW_X_DIR: now also J8.7; no longer J3.7
- net RW_X_OUTFG: now also J8.13; no longer J3.13
- net RW_X_SPEED_CTRL: now also J8.1; no longer J3.1
- net RW_Y_DIR: now also J8.9; no longer J3.9
- net RW_Y_OUTFG: now also J7.1; no longer J3.15
- net RW_Y_SPEED_CTRL: now also J8.3; no longer J3.3
- net RW_Z_DIR: now also J8.11; no longer J3.11
- net RW_Z_OUTFG: now also J7.2; no longer J3.16
- net RW_Z_SPEED_CTRL: now also J8.5; no longer J3.5
- net UCB0_SPI_CLK: now also J7.4; no longer J2.2
- net UCB0_SPI_MISO: now also J7.6; no longer J2.4
- net UCB0_SPI_MOSI: now also J7.8; no longer J2.6
Other:
- note removed: "3V3 Present Signal"
- note removed: "5V Present Signal"
