File: eagle projects/Z- Sun Sensor Board/ZMinusSunSensorBoard.brd (EAGLE design)
At the start: 91 x 91 mm, 189 parts, among them J2 HIROSE_FH19C-6S-0.5SH(10), J3 HIROSE_FH19C-6S-0.5SH(10), J4 HIROSE_FH19C-6S-0.5SH(10), J5 HIROSE_FH19C-6S-0.5SH(10), U1 ADS7841E_2K5, U13 ADS7841E_2K5, U15 TLV9051IDCKR, U19 TLV9051IDCKR, U2 ADS7841E_2K5, U21 TLV9051IDCKR, U23 TLV9051IDCKR, U24 TLV9051IDCKR, U25 ADS7841E_2K5, U26 TLV9051IDCKR, U27 ADS7841E_2K5, U28 TLV9051IDCKR, U29 TLV9051IDCKR, U3 TLV9051IDCKR, U30 TLV9051IDCKR, U31 TLV9051IDCKR, U32 TLV9051IDCKR, U4 LM20BIM7X_NOPB, U6 TLV9051IDCKR, U8 TLV9051IDCKR, U9 TLV9051IDCKR

Commit message: bfwebfibc
Parts:
- added R12, R16, R18, R21: 5.1M, rcl:R0402
- added R17: 5.1M, resistor:R0402
Connections:
- new net N$50: R12.2, U13.13
- new net N$51: R16.2, U25.13
- new net N$52: R18.2, U27.13
- new net N$53: R21.2, U1.13
- net GND: now also R12.1, R16.1, R17.1, R18.1, R21.1
- net N$2: now also R17.2
Changed lines of the file:
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@@
 <attribute name="VALUE" x="21.59" y="5.08" size="1.27" layer="28" rot="MR90"/>
+</element>
+<element name="R12" library="rcl" library_urn="urn:adsk.eagle:library:334" package="R0402" package3d_urn="urn:adsk.eagle:package:23547/3" value="5.1M" x="-3.175" y="-6.985" smashed="yes">
+<attribute name="NAME" x="-3.81" y="-6.35" size="1.27" layer="25"/>
+<attribute name="POPULARITY" value="34" x="-3.175" y="-6.985" size="1.778" layer="27" display="off"/>
+<attribute name="SPICEPREFIX" value="R" x="-3.175" y="-6.985" size="1.778" layer="27" display="off"/>
+<attribute name="VALUE" x="-3.81" y="-8.89" size="1.27" layer="27"/>
+</element>
+<element name="R16" library="rcl" library_urn="urn:adsk.eagle:library:334" package="R0402" package3d_urn="urn:adsk.eagle:package:23547/3" value="5.1M" x="-3.175" y="-12.065" smashed="yes">
+<attribute name="NAME" x="-3.81" y="-11.43" size="1.27" layer="25"/>
+<attribute name="POPULARITY" value="34" x="-3.175" y="-12.065" size="1.778" layer="27" display="off"/>
+<attribute name="SPICEPREFIX" value="R" x="-3.175" y="-12.065" size="1.778" layer="27" display="off"/>
+<attribute name="VALUE" x="-3.81" y="-13.97" size="1.27" layer="27"/>
+</element>
+<element name="R17" library="resistor" library_urn="urn:adsk.eagle:library:348" package="R0402" package3d_urn="urn:adsk.eagle:package:26058/2" value="5.1M" x="-2.54" y="-17.145" smashed="yes">
+<attribute name="NAME" x="-3.175" y="-16.51" size="1.27" layer="25"/>
+<attribute name="VALUE" x="-3.175" y="-19.05" size="1.27" layer="27"/>
+</element>
+<element name="R18" library="rcl" library_urn="urn:adsk.eagle:library:334" package="R0402" package3d_urn="urn:adsk.eagle:package:23547/3" value="5.1M" x="-3.175" y="-22.225" smashed="yes">
+<attribute name="NAME" x="-3.81" y="-21.59" size="1.27" layer="25"/>
+<attribute name="POPULARITY" value="34" x="-3.175" y="-22.225" size="1.778" layer="27" display="off"/>
+<attribute name="SPICEPREFIX" value="R" x="-3.175" y="-22.225" size="1.778" layer="27" display="off"/>
+<attribute name="VALUE" x="-3.81" y="-24.13" size="1.27" layer="27"/>
+</element>
+<element name="R21" library="rcl" library_urn="urn:adsk.eagle:library:334" package="R0402" package3d_urn="urn:adsk.eagle:package:23547/3" value="5.1M" x="-3.175" y="-27.305" smashed="yes">
+<attribute name="NAME" x="-3.81" y="-26.67" size="1.27" layer="25"/>
+<attribute name="POPULARITY" value="34" x="-3.175" y="-27.305" size="1.778" layer="27" display="off"/>
+<attribute name="SPICEPREFIX" value="R" x="-3.175" y="-27.305" size="1.778" layer="27" display="off"/>
+<attribute name="VALUE" x="-3.81" y="-29.21" size="1.27" layer="27"/>
 </element>
 </elements>
@@
 <contactref element="LED1" pad="C"/>
 <wire x1="26.035" y1="6.465" x2="26.035" y2="8.89" width="0.2032" layer="16"/>
+<contactref element="R12" pad="1"/>
+<contactref element="R16" pad="1"/>
+<contactref element="R17" pad="1"/>
+<contactref element="R18" pad="1"/>
+<contactref element="R21" pad="1"/>
 <wire x1="46.555" y1="86.0844" x2="47.555" y2="87.61" width="0" layer="19" extent="16-16"/>
 <wire x1="45.555" y1="85.11" x2="46.555" y2="85.11" width="0" layer="19" extent="16-16"/>
@@
 <wire x1="5.405" y1="46.48" x2="6.9306" y2="45.48" width="0" layer="19" extent="16-16"/>
 <wire x1="5.405" y1="41.98" x2="6.985" y2="43.4975" width="0" layer="19" extent="16-16"/>
+<wire x1="-3.675" y1="-6.985" x2="26.035" y2="6.465" width="0" layer="19" extent="1-16"/>
+<wire x1="-3.675" y1="-12.065" x2="-3.675" y2="-6.985" width="0" layer="19" extent="1-1"/>
+<wire x1="-3.19" y1="-17.145" x2="-3.675" y2="-12.065" width="0" layer="19" extent="1-1"/>
+<wire x1="-3.675" y1="-22.225" x2="-3.19" y2="-17.145" width="0" layer="19" extent="1-1"/>
+<wire x1="-3.675" y1="-27.305" x2="-3.675" y2="-22.225" width="0" layer="19" extent="1-1"/>
 </signal>
 <signal name="UCB0_SPI_CLK">
@@
 <contactref element="TP2" pad="1"/>
 <wire x1="66.9925" y1="12.7" x2="66.9925" y2="14.5923" width="0.2032" layer="16"/>
+<contactref element="R17" pad="2"/>
+<wire x1="-1.89" y1="-17.145" x2="66.9925" y2="12.7" width="0" layer="19" extent="1-1"/>
 </signal>
 <signal name="!CS!_SUN_X+">
@@
 <wire x1="23.595" y1="4.965" x2="23.495" y2="4.865" width="0.2032" layer="16"/>
 </signal>
+<signal name="N$50">
+<contactref element="U13" pad="13"/>
+<contactref element="R12" pad="2"/>
+<wire x1="-2.675" y1="-6.985" x2="83.5025" y2="14.5923" width="0" layer="19" extent="1-16"/>
+</signal>
+<signal name="N$51">
+<contactref element="U25" pad="13"/>
+<contactref element="R16" pad="2"/>
+<wire x1="-2.675" y1="-12.065" x2="58.7375" y2="14.5923" width="0" layer="19" extent="1-16"/>
+</signal>
+<signal name="N$52">
+<contactref element="R18" pad="2"/>
+<contactref element="U27" pad="13"/>
+<wire x1="-2.675" y1="-22.225" x2="50.4825" y2="14.5923" width="0" layer="19" extent="1-16"/>
+</signal>
+<signal name="N$53">
+<contactref element="U1" pad="13"/>
+<contactref element="R21" pad="2"/>
+<wire x1="-2.675" y1="-27.305" x2="75.2475" y2="14.5923" width="0" layer="19" extent="1-16"/>
+</signal>
 </signals>
