File: eagle projects/Z- Sun Sensor Board/ZMinusSunSensorBoard.sch (EAGLE design)
At the start: 189 parts, among them J2 HIROSE_FH19C-6S-0.5SH(10), J3 HIROSE_FH19C-6S-0.5SH(10), J4 HIROSE_FH19C-6S-0.5SH(10), J5 HIROSE_FH19C-6S-0.5SH(10), U1 ADS7841E_2K5, U13 ADS7841E_2K5, U15 TLV9051IDCKR, U19 TLV9051IDCKR, U2 ADS7841E_2K5, U21 TLV9051IDCKR, U23 TLV9051IDCKR, U24 TLV9051IDCKR, U25 ADS7841E_2K5, U26 TLV9051IDCKR, U27 ADS7841E_2K5, U28 TLV9051IDCKR, U29 TLV9051IDCKR, U3 TLV9051IDCKR, U30 TLV9051IDCKR, U31 TLV9051IDCKR, U32 TLV9051IDCKR, U4 LM20BIM7X_NOPB, U6 TLV9051IDCKR, U8 TLV9051IDCKR, U9 TLV9051IDCKR

Commit message: bfwebfibc
Parts:
- added R12, R16, R18, R21: 5.1M, rcl:R-US_R0402
- added R17: 5.1M, resistor:R-US_R0402
Connections:
- new net N$50: R12.2, U13.BUSY
- new net N$51: R16.2, U25.BUSY
- new net N$52: R18.2, U27.BUSY
- new net N$53: R21.2, U1.BUSY
- net GND: now also R12.1, R16.1, R17.1, R18.1, R21.1
- net N$2: now also R17.2
Other:
- note added: "Thomas Christison"
- moved on the sheet: C102, C22, C51, C81, C95, R10, R5
